File: Campinglaterne.kicad_pcb (KiCad board)
At the start: 2 copper layers, 67.9 x 67.5 mm, 160 parts, among them J1 USB_C_Receptacle_USB2.0, J10 Conn_01x02_Female, J11 Conn_01x02_Female, J12 Conn_01x02_Female, J13 Conn_01x02_Female, J14 Conn_01x02_Female, J15 Conn_01x02_Female, J16 Conn_01x02_Female, J17 Conn_01x02_Female, J2 Conn_01x02_Female, J3 Conn_01x02_Female, J4 Conn_01x02_Female, J5 Conn_01x02_Female, J6 Conn_01x02_Female, J7 Conn_01x02_Female, J8 Conn_01x02_Female, J9 Conn_01x02_Female, Q1 Q_NPN_BEC, Q10 Q_NPN_BEC, Q11 Q_NPN_BEC, Q12 Q_NPN_BEC, Q13 Q_NPN_BEC, Q14 Q_NPN_BEC, Q2 Q_NPN_BEC, Q3 SSM3J358R,LF, Q4 Q_NPN_BEC, Q5 Q_NPN_BEC, Q6 SSM3J358R,LF, Q7 SSM3J358R,LF, Q8 Q_NPN_BEC, Q9 Q_NPN_BEC, U1 ISL80015, U2 BD48K30G-TL, U3 FAN48610, U4 BD48K35G-TL, U5 4017, U6 MCP1664, U7 SA555DR, U8 AZV321KSTR-G1, U9 TL431DBZ

Commit message: Add files via upload
Routing:
- net Net-(C26-Pad1): track 54.1 -> 53.5 mm, vias 8 -> 2
Changed lines of the file:
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@@
   (segment (start 132.35 97.05) (end 131.6 97.8) (width 0.25) (layer "F.Cu") (net 68))
   (segment (start 132.1 90.925) (end 132.1 91.25) (width 0.25) (layer "F.Cu") (net 68))
-  (segment (start 126.25 103.725) (end 125.9 103.375) (width 1) (layer "F.Cu") (net 68))
   (segment (start 135.9 95.9) (end 136.4125 95.3875) (width 2) (layer "F.Cu") (net 68))
   (segment (start 140.170592 96.60048) (end 140.071552 96.69952) (width 0.25) (layer "F.Cu") (net 68))
@@
   (segment (start 126.25 103.725) (end 126.25 106.475) (width 1) (layer "F.Cu") (net 68))
   (segment (start 141.852618 96.60048) (end 140.170592 96.60048) (width 0.25) (layer "F.Cu") (net 68))
-  (segment (start 126.25 103.225) (end 123.925 100.9) (width 1.5) (layer "F.Cu") (net 68))
   (segment (start 130.16202 109.07452) (end 129.9 108.8125) (width 2) (layer "F.Cu") (net 68))
   (segment (start 122.1 100.9) (end 122.1 100.7) (width 1) (layer "F.Cu") (net 68))
   (segment (start 126.9375 108.8125) (end 126.625 108.5) (width 0.5) (layer "F.Cu") (net 68))
+  (segment (start 126.25 103.437263) (end 122.412737 99.6) (width 2) (layer "F.Cu") (net 68))
   (segment (start 120 97.475) (end 120 99.5) (width 0.25) (layer "F.Cu") (net 68))
   (segment (start 132.35 95.9) (end 132.35 97.05) (width 0.25) (layer "F.Cu") (net 68))
@@
   (segment (start 123 98.65) (end 122.05 99.6) (width 1.5) (layer "F.Cu") (net 68))
   (segment (start 126.575 108.45) (end 126.625 108.5) (width 0.25) (layer "F.Cu") (net 68))
+  (segment (start 122.412737 99.6) (end 122.05 99.6) (width 2) (layer "F.Cu") (net 68))
   (segment (start 120.95 99.75) (end 122.1 100.9) (width 1) (layer "F.Cu") (net 68))
   (segment (start 132.1 91.25) (end 131.7 91.65) (width 0.25) (layer "F.Cu") (net 68))
@@
   (segment (start 142.3 97.047862) (end 141.852618 96.60048) (width 0.25) (layer "F.Cu") (net 68))
   (segment (start 126.25 106.475) (end 126.575 106.8) (width 1) (layer "F.Cu") (net 68))
-  (via (at 122.25 100.85) (size 0.8) (drill 0.4) (layers "F.Cu" "B.Cu") (net 68))
-  (via (at 121.5 100.3) (size 0.8) (drill 0.4) (layers "F.Cu" "B.Cu") (net 68))
+  (segment (start 126.25 103.725) (end 126.25 103.437263) (width 2) (layer "F.Cu") (net 68))
   (via (at 131.7 91.65) (size 0.8) (drill 0.4) (layers "F.Cu" "B.Cu") (net 68))
   (via (at 132.4625 93.9) (size 0.8) (drill 0.4) (layers "F.Cu" "B.Cu") (net 68))
-  (via (at 124.25 102.05) (size 0.8) (drill 0.4) (layers "F.Cu" "B.Cu") (net 68))
-  (via (at 124.6 101) (size 0.8) (drill 0.4) (layers "F.Cu" "B.Cu") (net 68))
-  (via (at 122.3 99.75) (size 0.8) (drill 0.4) (layers "F.Cu" "B.Cu") (net 68))
-  (via (at 123.5 101.35) (size 0.8) (drill 0.4) (layers "F.Cu" "B.Cu") (net 68))
-  (segment (start 124.3 101.5) (end 123.1 100.3) (width 2) (layer "B.Cu") (net 68))
   (segment (start 131.7 91.65) (end 131.7 93.1375) (width 0.25) (layer "B.Cu") (net 68))
   (segment (start 131.7 93.1375) (end 132.4625 93.9) (width 0.25) (layer "B.Cu") (net 68))
-  (segment (start 123.1 100.3) (end 121.9 100.3) (width 2) (layer "B.Cu") (net 68))
   (segment (start 171.975 102.0875) (end 172.05 102.1625) (width 0.25) (layer "F.Cu") (net 69))
   (segment (start 172.05 102.3) (end 170.45 103.9) (width 0.25) (layer "F.Cu") (net 69))
@@
       )
     )
-  )
-  (zone (net 68) (net_name "Net-(C26-Pad1)") (layer "F.Cu") (hatch edge 0.508)
-    (priority 5)
-    (connect_pads yes (clearance 0.25))
-    (min_thickness 0.254) (filled_areas_thickness no)
-    (fill yes (thermal_gap 0.508) (thermal_bridge_width 0.508))
-    (polygon
-      (pts
-        (xy 127.45 101.65)
-        (xy 127.45 103.75)
-        (xy 122.9 103.75)
-        (xy 122.9 100.5)
-        (xy 123.75 99.65)
-        (xy 125.05 99.65)
-        (xy 125.25 99.45)
-      )
-    )
