File: Campinglaterne.kicad_sch (KiCad schematic)
At the start: 160 parts, among them J1 USB_C_Receptacle_USB2.0, J10 Conn_01x02_Female, J11 Conn_01x02_Female, J12 Conn_01x02_Female, J13 Conn_01x02_Female, J14 Conn_01x02_Female, J15 Conn_01x02_Female, J16 Conn_01x02_Female, J2 Conn_01x02_Female, J3 Conn_01x02_Female, J4 Conn_01x02_Female, J5 Conn_01x02_Female, J6 Conn_01x02_Female, J7 Conn_01x02_Female, J8 Conn_01x02_Female, J9 Conn_01x02_Female, Q1 Q_NPN_BEC, Q10 Q_NPN_BEC, Q11 Q_NPN_BEC, Q12 Q_NPN_BEC, Q13 Q_NPN_BEC, Q14 Q_NPN_BEC, Q2 Q_NPN_BEC, Q3 SSM3J358R,LF, Q4 Q_NPN_BEC, Q5 Q_NPN_BEC, Q6 SSM3J358R,LF, Q7 SSM3J358R,LF, Q8 Q_NPN_BEC, Q9 Q_NPN_BEC, U1 ISL80015, U2 BD48K30G-TL, U3 FAN48610, U4 BD48K35G-TL, U5 4017, U6 MCP1664, U7 SA555DR, U8 AZV321KSTR-G1, U9 TL431DBZ

Commit message: Add files via upload
Parts:
- gave numbers to parts that had none: 3
Changed lines of the file:
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@@
   (symbol (lib_id "Device:LED") (at 101.6 287.02 90) (unit 1)
     (in_bom yes) (on_board yes)
-    (property "Reference" "D?" (id 0) (at 102.87 284.48 90)
+    (property "Reference" "D5" (id 0) (at 102.87 284.48 90)
       (effects (font (size 1.27 1.27)) (justify right))
     )
@@
   (symbol (lib_id "Device:R") (at 101.6 276.86 0) (unit 1)
     (in_bom yes) (on_board yes) (fields_autoplaced)
-    (property "Reference" "R?" (id 0) (at 103.378 276.0253 0)
+    (property "Reference" "R58" (id 0) (at 103.378 276.0253 0)
       (effects (font (size 1.27 1.27)) (justify left))
     )
@@
   (symbol (lib_id "Connector:Conn_01x02_Female") (at 111.76 287.02 0) (unit 1)
     (in_bom yes) (on_board yes) (fields_autoplaced)
-    (property "Reference" "J?" (id 0) (at 112.4712 287.4553 0)
+    (property "Reference" "J17" (id 0) (at 112.4712 287.4553 0)
       (effects (font (size 1.27 1.27)) (justify left))
     )
@@
       (reference "D4") (unit 1) (value "15V") (footprint "Diode_SMD:D_SOT-23_ANK")
     )
+    (path "/21d64de5-121d-4912-9a18-ef086f5b44bc"
+      (reference "D5") (unit 1) (value "LED yellow") (footprint "LED_SMD:LED_0603_1608Metric")
+    )
     (path "/4f48ff2e-9390-47df-9a1b-dc8aefe60ddd"
       (reference "D6") (unit 1) (value "D_Schottky") (footprint "Diode_SMD:D_SMB")
@@
       (reference "D11") (unit 1) (value "LED orange") (footprint "LED_SMD:LED_0603_1608Metric")
     )
-    (path "/21d64de5-121d-4912-9a18-ef086f5b44bc"
-      (reference "D?") (unit 1) (value "LED yellow") (footprint "LED_SMD:LED_0603_1608Metric")
-    )
     (path "/85350319-8ae0-4928-abe3-2ebd069ba920"
       (reference "H1") (unit 1) (value "MountingHole") (footprint "MountingHole:MountingHole_3.2mm_M3_ISO14580")
@@
     )
     (path "/e31e9de9-33a9-47a1-ba4c-67658a743fa1"
-      (reference "J?") (unit 1) (value "Conn_01x02_Female") (footprint "Connector_PinSocket_2.54mm:PinSocket_1x02_P2.54mm_Vertical")
+      (reference "J17") (unit 1) (value "Conn_01x02_Female") (footprint "Connector_PinSocket_2.54mm:PinSocket_1x02_P2.54mm_Vertical")
     )
     (path "/f53938da-cdab-4f71-91f4-ea7fc2466c96"
@@
       (reference "R57") (unit 1) (value "10k") (footprint "Resistor_SMD:R_0603_1608Metric")
     )
+    (path "/9ca7c142-8976-4bce-9681-5f8ed596edf1"
+      (reference "R58") (unit 1) (value "not_ass_1k") (footprint "Resistor_SMD:R_0603_1608Metric")
+    )
     (path "/0d9478b9-9d63-47f6-812d-b680b3b02598"
       (reference "R61") (unit 1) (value "10R") (footprint "Resistor_SMD:R_0603_1608Metric")
@@
       (reference "R62") (unit 1) (value "10R") (footprint "Resistor_SMD:R_0603_1608Metric")
     )
-    (path "/9ca7c142-8976-4bce-9681-5f8ed596edf1"
-      (reference "R?") (unit 1) (value "not_ass_1k") (footprint "Resistor_SMD:R_0603_1608Metric")
-    )
     (path "/657f9c17-1432-414d-b1e4-85e6f3e98841"

Commit message: Add files via upload
Parts:
- C2: Config (none) -> +Dev
- D11, D5, L1, U6: Config (none) -> -Rel
Changed lines of the file:
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@@
+      (effects (font (size 1.27 1.27)) hide)
+    )
+    (property "Config" "-Rel" (id 4) (at 669.29 163.83 0)
       (effects (font (size 1.27 1.27)) hide)
     )
@@
     )
     (property "Datasheet" "~" (id 3) (at 101.6 287.02 0)
+      (effects (font (size 1.27 1.27)) hide)
+    )
+    (property "Config" "-Rel" (id 4) (at 101.6 287.02 0)
       (effects (font (size 1.27 1.27)) hide)
     )
@@
       (effects (font (size 1.27 1.27)) hide)
     )
+    (property "Config" "-Rel" (id 4) (at 165.1 275.59 0)
+      (effects (font (size 1.27 1.27)) hide)
+    )
     (pin "1")
     (pin "2")
@@
     )
     (property "Datasheet" "~" (id 3) (at 612.14 430.53 0)
+      (effects (font (size 1.27 1.27)) hide)
+    )
+    (property "Config" "-Rel" (id 4) (at 612.14 430.53 0)
       (effects (font (size 1.27 1.27)) hide)
     )
@@
       (effects (font (size 1.27 1.27)) hide)
     )
+    (property "Config" "+Dev" (id 4) (at 182.88 281.94 0)
+      (effects (font (size 1.27 1.27)) hide)
+    )

Commit message: Add files via upload
Parts:
- C2: Config +Dev -> +DEV
- D11, D5, L1, U6: Config -Rel -> -REL
Changed lines of the file:
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@@
       (effects (font (size 1.27 1.27)) hide)
     )
-    (property "Config" "-Rel" (id 4) (at 669.29 163.83 0)
+    (property "Config" "-REL" (id 4) (at 669.29 163.83 0)
       (effects (font (size 1.27 1.27)) hide)
     )
@@
       (effects (font (size 1.27 1.27)) hide)
     )
-    (property "Config" "-Rel" (id 4) (at 101.6 287.02 0)
+    (property "Config" "-REL" (id 4) (at 101.6 287.02 0)
       (effects (font (size 1.27 1.27)) hide)
     )
@@
       (effects (font (size 1.27 1.27)) hide)
     )
-    (property "Config" "-Rel" (id 4) (at 165.1 275.59 0)
+    (property "Config" "-REL" (id 4) (at 165.1 275.59 0)
       (effects (font (size 1.27 1.27)) hide)
     )
@@
       (effects (font (size 1.27 1.27)) hide)
     )
-    (property "Config" "-Rel" (id 4) (at 612.14 430.53 0)
+    (property "Config" "-REL" (id 4) (at 612.14 430.53 0)
       (effects (font (size 1.27 1.27)) hide)
     )
@@
       (effects (font (size 1.27 1.27)) hide)
     )
-    (property "Config" "+Dev" (id 4) (at 182.88 281.94 0)
+    (property "Config" "+DEV" (id 4) (at 182.88 281.94 0)
       (effects (font (size 1.27 1.27)) hide)
     )

Commit message: Add files via upload
Parts:
- C1, C10, C11, C12, C13, C14, C15, C18, C20, C21, C22, C23, C24, C26, C27, C3, C4, C5, C6, C7, C8, C9, D1, D10, D2, D3, D4, D6, D7, D8, D9, H1, H2, H3, J1, J10, J11, J12, J13, J14, J15, J16, J17, J2, J3, J4, J5, J6, J7, J8, J9, JP2, L3, Q1, Q10, Q11, Q12, Q13, Q14, Q2, Q3, Q4, Q5, Q6, Q7, Q8, Q9, R1, R10, R12, R13, R15, R16, R18, R19, R2, R20, R21, R22, R23, R24, R25, R26, R27, R28, R29, R3, R30, R31, R32, R33, R34, R35, R36, R37, R38, R39, R4, R41, R42, R43, R45, R46, R47, R48, R49, R5, R50, R51, R53, R54, R55, R56, R57, R58, R6, R7, R8, R9, U1, U2, U3, U5, U7, U8: Config (none) -> +DEV
- L4, R11, R14, R17, R40, R44, R52, R61, R62, TP1, TP10, TP11, TP12, TP13, TP14, TP15, TP16, TP17, TP18, TP19, TP2, TP3, TP4, TP5, TP6, TP7, TP8, TP9, U4, U9: Config (none) -> -REL
- U6: Config -REL -> +DEV

Commit message: Add files via upload
Parts:
- J1, U1, U5: Config +DEV -> +DEV,+REL
Changed lines of the file:
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@@
       (effects (font (size 1.27 1.27)) hide)
     )
-    (property "Config" "+DEV" (id 4) (at 588.01 309.88 0)
+    (property "Config" "+DEV,+REL" (id 4) (at 588.01 309.88 0)
       (effects (font (size 1.27 1.27)) hide)
     )
@@
       (effects (font (size 1.27 1.27)) hide)
     )
-    (property "Config" "+DEV" (id 4) (at 143.51 280.67 0)
+    (property "Config" "+DEV,+REL" (id 4) (at 143.51 280.67 0)
       (effects (font (size 1.27 1.27)) hide)
     )
@@
       (effects (font (size 1.27 1.27)) hide)
     )
-    (property "Config" "+DEV" (id 4) (at 57.15 273.05 0)
-      (effects (font (size 1.27 1.27)) hide)
-    )
+    (property "Config" "+DEV,+REL" (id 4) (at 57.15 273.05 0)
+      (effects (font (size 1.27 1.27)) hide)
+    )

Commit message: Add files via upload
Parts:
- C1, C10, C11, C13, C15, C20, C24, C26, C3, C4, C5, C8, D1, D10, D2, D3, D6, D8, D9, H1, H2, H3, J10, J11, J12, J13, J14, J15, J16, J17, J2, J3, J4, J5, J6, J7, J8, J9, JP2, L3, Q1, Q10, Q11, Q12, Q13, Q14, Q2, Q3, Q4, Q5, Q6, Q7, Q8, Q9, R1, R10, R12, R13, R15, R16, R18, R19, R2, R20, R21, R22, R23, R24, R25, R26, R27, R28, R29, R3, R30, R31, R32, R33, R34, R35, R36, R37, R38, R39, R4, R41, R42, R43, R45, R46, R47, R48, R49, R5, R50, R51, R53, R54, R55, R56, R57, R58, R6, R7, R8, R9, U2, U3, U6, U7, U8: Config +DEV -> (none)
- C12, C18: Config +DEV -> -REL
- C14, C27: Config +DEV -> +REL
- C21, C22, C23, C6, C7, C9: Config +DEV -> -DEV
- D11: Config -REL -> -REL,+DEV
- D4, D7: Config +DEV -> -REL,-DEV
- D5: Config -REL -> -DEV,+REL
- J1, U1, U5: Config +DEV,+REL -> (none)
- L1, L4, R11, R14, R17, R40, R44, R52, R61, R62, TP1, TP10, TP11, TP12, TP13, TP14, TP15, TP16, TP17, TP18, TP19, TP2, TP3, TP4, TP5, TP6, TP7, TP8, TP9, U4, U9: Config -REL -> (none)

Commit message: Add files via upload
Parts:
- C14, C27: REL:Value (none) -> 10µ 1000V
Changed lines of the file:
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@@
+      (effects (font (size 1.27 1.27)) hide)
+    )
+    (property "REL:Value" "10µ 1000V" (id 5) (at 703.58 149.86 0)
       (effects (font (size 1.27 1.27)) hide)
     )
@@
       (effects (font (size 1.27 1.27)) hide)
     )
+    (property "REL:Value" "10µ 1000V" (id 5) (at 697.23 149.86 0)
+      (effects (font (size 1.27 1.27)) hide)
+    )
